Commit message: minor changes

File: tests/data/kuka_iiwa/fixed_joint_4.urdf (robot description, URDF)
Before this commit: robot lbr_iiwa, 8 links, 7 joints
Links:
- link lbr_iiwa_link_0: mass 0.0 -> 5.0

File: tests/data/kuka_iiwa/model.urdf (robot description, URDF)
Before this commit: robot lbr_iiwa, 8 links, 7 joints
Links:
- link lbr_iiwa_link_0: mass 0.0 -> 5.0
